File: Schematic/Minimal/kicad/SDMin.kicad_pcb (KiCad board)
At the start: 2 copper layers, 85 parts, among them CON1 uSD_Card, P1 USB_B, P2 CONN_01X04, P3 CONN_01X04, P4 CONN_01X04, SW1 SW_PUSH, SW2 SW_PUSH, SW3 SW_PUSH, SW4 SW_PUSH, SW5 Switch_SPDT_x2, SW6 SW_PUSH, SW7 SW_PUSH, SW8 SW_PUSH, SW9 SW_PUSH, U1 AAT1217, U10 ADMP401-BB, U11 RN-52, U12 STA013, U2 PAM2301, U3 MCP73811/2, U4 STM32L476R, U5 Lightware_SF10/A, U6 UART, U7 DebugPins, U8 MLX90393, U9 LS20031, X1 14.7456MHz

Commit message: Working on the PCB (third attempt). Misc schematic fixes (charger always on)
Parts:
- removed R20: 1M, Resistors_SMD:R_0805_HandSoldering
- removed R21: 470, Resistors_SMD:R_0805_HandSoldering
- removed R22: 47, Resistors_SMD:R_0805_HandSoldering
- added REF**: LaserHolder, con-trougnouf:LaserHolder, F.Cu at (198.0, 76.6)
- C10: value 10uF -> 4.7uF
- C11: value 0.1uF -> 10uF; footprint Capacitors_SMD:C_0805_HandSoldering -> Capacitors_ThroughHole:C_Radial_D5_L11_P2.5
- C12, C14, C16, C5: value 4.7uF -> 0.1uF; footprint Capacitors_ThroughHole:C_Radial_D5_L11_P2.5 -> Capacitors_SMD:C_0805_HandSoldering; moved to B.Cu
- C13, C15: value 0.1uF -> 4.7uF; footprint Capacitors_SMD:C_0805_HandSoldering -> Capacitors_ThroughHole:C_Radial_D5_L11_P2.5
- C17: value 47uF -> 4.7uF
- C18: value 0.1uF -> 47uF; footprint Capacitors_SMD:C_0805_HandSoldering -> Capacitors_ThroughHole:C_Radial_D5_L11_P2.5
- C19, C20, C24, C25, C29, C4, R1, R12, R13, R3, R5, R6, R8, X1: moved to B.Cu
- C2: value 1uF -> 4.7uF; footprint Capacitors_ThroughHole:C_Radial_D5_L11_P2.5 -> Capacitors_SMD:C_0805_HandSoldering
- C26: value 470pF -> 0.1uF; moved to B.Cu
- C27: value 4.7nF -> 470pF; moved to B.Cu
- C28: value 22pF -> 4.7nF; moved to B.Cu
- C3, C8: value 4.7uF -> 1uF
- C30: value 0.1uF -> 22pF; moved to B.Cu
- C7: value 0.1uF -> 10uF
- C9: value 1uF -> 0.1uF; footprint Capacitors_ThroughHole:C_Radial_D5_L11_P2.5 -> Capacitors_SMD:C_0805_HandSoldering; moved to B.Cu
- R10, R11, R9: value 10K -> 47K; moved to B.Cu
- R14, R15: value 47K -> 4.7; moved to B.Cu
- R16: value 47K -> 1k; moved to B.Cu
- R17: value 4.7 -> 1M; moved to B.Cu
- R18: value 4.7 -> 470
- R19: value 1k -> 47
- R2: value 332k -> 10K; moved to B.Cu
- R4: value 1.02M -> 10K; moved to B.Cu
- R7: value 1M -> 10K; moved to B.Cu
- U1: value AAT1217 -> PAM2301; footprint TO_SOT_Packages_SMD:SOT-23-6 -> TO_SOT_Packages_SMD:SOT-23-5
- U10: footprint Pin_Headers:Pin_Header_Straight_1x03 -> con-trougnouf:INMP401-bb
- U2: value PAM2301 -> XC9140
- U7: footprint Pin_Headers:Pin_Header_Straight_1x05 -> Pin_Headers:Pin_Header_Straight_1x04
- U9: footprint Pin_Headers:Pin_Header_Straight_1x05 -> con-trougnouf:LS20031+H
- moved P2 234.7 mm to (227.4, 128.3), turned to 180 degrees
- moved R8 231.2 mm to (243.7, 158.8), turned to 180 degrees
- moved R1 231.1 mm to (253.7, 158.8)
- moved U10 219.8 mm to (246.0, 110.0), turned to 180 degrees
- moved P3 216.2 mm to (224.9, 128.3), turned to 180 degrees
- moved SW1 216.0 mm to (253.7, 158.8)
- moved R3 209.6 mm to (224.0, 158.5)
- moved U9 206.1 mm to (226.2, 82.8)
- moved SW9 204.8 mm to (243.8, 158.7)
- moved P4 204.1 mm to (222.3, 128.3), turned to 180 degrees
- moved R5 204.0 mm to (203.9, 158.6)
- moved R7 197.3 mm to (234.0, 158.5), turned to 180 degrees
- moved R2 190.0 mm to (214.0, 158.5)
- moved C18 173.6 mm to (190.4, 88.8), turned to 90 degrees
- moved R4 171.1 mm to (193.9, 158.6)
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Connections:
- C10 pad 1: Net-(C10-Pad1) -> GND
- C10 pad 2: GND -> +3V3
- C18 pad 1: +3V3 -> GND
- C18 pad 2: GND -> +3V3
- C19 pad 1: Net-(C19-Pad1) -> +3V3
- C19 pad 2: +3V3 -> GND
- C2 pad 1: GND -> +BATT
- C2 pad 2: Net-(C2-Pad2) -> GND
- C20 pad 1: Net-(C19-Pad1) -> GND
- C25 pad 1: Net-(C25-Pad1) -> GND
- C25 pad 2: Net-(C25-Pad2) -> +3V3
- C26 pad 2: GND -> Net-(C26-Pad2)
- C3 pad 2: +5V -> Net-(C3-Pad2)
- C30 pad 1: GND -> Net-(C30-Pad1)
- C30 pad 2: +3V3 -> GND
- C6 pad 1: +BATT -> GND
- C6 pad 2: GND -> +3V3
- C7 pad 1: GND -> +5V
- C7 pad 2: +3V3 -> GND
- C8 pad 1: GND -> Net-(BT1-Pad1)
- C8 pad 2: +3V3 -> GND
- C9 pad 1: +BATT -> GND
- C9 pad 2: GND -> +3V3
- L1 pad 1: Net-(L1-Pad1) -> +BATT
- L1 pad 2: +BATT -> Net-(L1-Pad2)
- P1 pad 1: Net-(C2-Pad2) -> Net-(C3-Pad2)
- P1 pad 2: Net-(P1-Pad2) -> (no net)
- P1 pad 3: Net-(P1-Pad3) -> (no net)
- P1 pad 5: Net-(P1-Pad5) -> (no net)
- P2 pad 3: Net-(P2-Pad3) -> (no net)
- P4 pad 3: Net-(P4-Pad3) -> (no net)
- R10 pad 1: GND -> PC8_SD-D0
- R10 pad 2: /in3 -> +3V3
- R11 pad 1: GND -> PD2_SD-CMD
- R11 pad 2: /in4 -> +3V3
- R12 pad 1: PC9_SD-D1 -> +3V3
- R12 pad 2: +3V3 -> PC11_SD-D3
- R13 pad 1: PC8_SD-D0 -> +3V3
- R13 pad 2: +3V3 -> PC10_SD-D2
- R14 pad 1: PD2_SD-CMD -> +3V3
- R14 pad 2: +3V3 -> Net-(C26-Pad2)
- R15 pad 1: +3V3 -> GND
- R15 pad 2: PC11_SD-D3 -> Net-(C26-Pad1)
- R16 pad 1: +3V3 -> Net-(C27-Pad1)
- R16 pad 2: PC10_SD-D2 -> Net-(C28-Pad1)
- R17 pad 1: +3V3 -> Net-(C30-Pad1)
- R17 pad 2: Net-(C25-Pad2) -> Net-(C29-Pad1)
- R18 pad 1: GND -> +3V3
- R18 pad 2: Net-(C25-Pad1) -> Net-(D3-Pad2)
- R19 pad 1: Net-(C26-Pad1) -> +3V3
- R19 pad 2: Net-(C27-Pad1) -> Net-(D2-Pad2)
- R2 pad 1: Net-(R2-Pad1) -> GND
- R2 pad 2: GND -> /in6
- R3 pad 2: /in6 -> /in7
- R4 pad 1: +5V -> GND
- R4 pad 2: Net-(R2-Pad1) -> /in8
- R5 pad 2: /in7 -> /in1
- R6 pad 2: /in8 -> /in2
- R7 pad 1: +BATT -> GND
- R7 pad 2: Net-(R7-Pad2) -> /in3
- R8 pad 2: /in1 -> /in4
- R9 pad 1: GND -> PC9_SD-D1
- R9 pad 2: /in2 -> +3V3
- SW5 pad 1: Net-(SW5-Pad1) -> (no net)
- U1 pad 1: Net-(L1-Pad1) -> +BATT
- U1 pad 3: Net-(R2-Pad1) -> Net-(L2-Pad1)
- U1 pad 4: Net-(R7-Pad2) -> +BATT
- U1 pad 5: +5V -> +3V3
- U11 pad 10: Net-(U11-Pad10) -> (no net)
- U11 pad 12: Net-(U11-Pad12) -> (no net)
- U11 pad 13: Net-(U11-Pad13) -> (no net)
- U11 pad 19: Net-(U11-Pad19) -> (no net)
- U11 pad 28: Net-(U11-Pad28) -> (no net)
- U11 pad 29: Net-(U11-Pad29) -> (no net)
- U11 pad 3: Net-(U11-Pad3) -> (no net)
- U11 pad 30: Net-(U11-Pad30) -> (no net)
- U11 pad 31: Net-(U11-Pad31) -> (no net)
- U11 pad 34: Net-(U11-Pad34) -> (no net)
- U11 pad 35: Net-(U11-Pad35) -> (no net)
- U11 pad 36: Net-(U11-Pad36) -> (no net)
- U11 pad 37: Net-(U11-Pad37) -> (no net)
- U11 pad 38: Net-(U11-Pad38) -> (no net)
- U11 pad 4: Net-(U11-Pad4) -> (no net)
- U11 pad 40: Net-(U11-Pad40) -> (no net)
- U11 pad 41: Net-(U11-Pad41) -> (no net)
- U11 pad 42: Net-(U11-Pad42) -> (no net)
- U11 pad 43: Net-(U11-Pad43) -> (no net)
- U11 pad 5: Net-(U11-Pad5) -> (no net)
- U11 pad 6: Net-(U11-Pad6) -> (no net)
- U11 pad 7: Net-(U11-Pad7) -> (no net)
- U11 pad 8: Net-(U11-Pad8) -> (no net)
- U11 pad 9: Net-(U11-Pad9) -> (no net)
- U12 pad 12: Net-(U12-Pad12) -> (no net)
- U12 pad 17: Net-(C25-Pad2) -> Net-(C26-Pad2)
- U12 pad 18: Net-(C25-Pad1) -> Net-(C26-Pad1)
- U12 pad 19: Net-(C26-Pad1) -> Net-(C27-Pad1)
- U12 pad 20: Net-(C28-Pad1) -> Net-(C29-Pad1)
- U12 pad 21: Net-(C29-Pad1) -> Net-(C30-Pad1)
- U2 pad 3: Net-(L2-Pad1) -> +BATT
- U2 pad 4: +BATT -> +5V
- U2 pad 5: +3V3 -> Net-(L1-Pad2)
- U3 pad 1: Net-(C2-Pad2) -> Net-(C3-Pad2)
- U3 pad 2: Net-(U3-Pad2) -> GND
- U3 pad 3: Net-(U3-Pad3) -> Net-(BT1-Pad1)
- U3 pad 4: Net-(C2-Pad2) -> Net-(C3-Pad2)
- U3 pad 5: Net-(C2-Pad2) -> Net-(C3-Pad2)
- U4 pad 38: Net-(U4-Pad38) -> (no net)
- U4 pad 56: Net-(U4-Pad56) -> (no net)
- U4 pad 58: Net-(U4-Pad58) -> (no net)
- U4 pad 60: Net-(U4-Pad60) -> (no net)
- U4 pad 61: Net-(U4-Pad61) -> (no net)
- U8 pad 13: Net-(C19-Pad1) -> GND
- X1 pad 1: Net-(C28-Pad1) -> Net-(C29-Pad1)
- X1 pad 2: Net-(C29-Pad1) -> Net-(C30-Pad1)
Routing:
- net (no net): track 0.00 -> 1107.0 mm, vias 0 -> 31
- net +3V3: track 0.00 -> 204.4 mm, vias 0 -> 7
- net GND: track 0.00 -> 146.1 mm, vias 0 -> 12
- net Net-(BT1-Pad1): track 0.00 -> 63.4 mm
- net +BATT: track 0.00 -> 60.4 mm
- net PC9_SD-D1: track 0.00 -> 56.7 mm, vias 0 -> 2
- net PC12_SD-CK: track 0.00 -> 53.2 mm
- net PC8_SD-D0: track 0.00 -> 51.0 mm, vias 0 -> 2
- net PD2_SD-CMD: track 0.00 -> 49.1 mm, vias 0 -> 2
- net PC10_SD-D2: track 0.00 -> 48.2 mm, vias 0 -> 2
- net PC11_SD-D3: track 0.00 -> 48.2 mm, vias 0 -> 2
- net PA15_SD-DET: track 0.00 -> 38.5 mm, vias 0 -> 2
- net Net-(C30-Pad1): track 0.00 -> 32.2 mm, vias 0 -> 1
- net PB7_GPS-TX: track 0.00 -> 29.4 mm, vias 0 -> 1
- net Net-(C29-Pad1): track 0.00 -> 27.3 mm, vias 0 -> 1
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- added copper zone on F.Cu, net +3V3
- added copper zone on B.Cu, net GND
Other:
- board outline added: 95 x 99 mm

Commit message: Slight progress on PCB attempt 3
Routing:
- net PB14_MP3-RST: track 0.00 -> 59.7 mm, vias 0 -> 2
- net PC6_MP3-DR: track 0.00 -> 54.4 mm, vias 0 -> 2
- net PA7_MP3-SDI: track 0.00 -> 43.8 mm
- net PA5_MP3-SCK: track 0.00 -> 42.3 mm
- net PB15_MAG-MOSI: track 0.00 -> 37.0 mm, vias 0 -> 2
- net Net-(P4-Pad1): track 0.00 -> 21.8 mm, vias 0 -> 1
- net Net-(P4-Pad2): track 0.00 -> 20.6 mm, vias 0 -> 1
- net Net-(P4-Pad4): track 0.00 -> 13.0 mm, vias 0 -> 1
Changed lines of the file:
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@@
-(kicad_pcb (version 4) (host pcbnew 4.0.2-stable)
+(kicad_pcb (version 4) (host pcbnew 4.0.1-stable)
   (general
     (links 257)
-    (no_connects 138)
-    (area 38.924999 55.924999 134.075001 155.075001)
+    (no_connects 130)
+    (area 24.149999 55.924999 265.000001 205.200002)
     (thickness 1.6)
     (drawings 11)
-    (tracks 877)
+    (tracks 960)
     (zones 0)
     (modules 83)
@@
   (layers
     (0 F.Cu signal)
-    (31 B.Cu signal hide)
+    (31 B.Cu signal)
     (32 B.Adhes user)
     (33 F.Adhes user)
@@
     (pad_to_mask_clearance 0.2)
     (aux_axis_origin 0 0)
-    (visible_elements FFFEFF7F)
+    (visible_elements FFFFFF7F)
     (pcbplotparams
       (layerselection 0x00030_80000001)
@@
   (segment (start 184.6 119.7) (end 184.6 116) (width 0.5) (layer F.Cu) (net 13))
   (segment (start 184.85 119.95) (end 184.6 119.7) (width 0.5) (layer F.Cu) (net 13))
+  (segment (start 213.9 119.705) (end 220.095 119.705) (width 0.25) (layer F.Cu) (net 33) (status 400000))
+  (segment (start 207.25 102.95) (end 207.25 96.7) (width 0.25) (layer F.Cu) (net 33) (status 800000))
+  (segment (start 207.2 103) (end 207.25 102.95) (width 0.25) (layer F.Cu) (net 33))
+  (segment (start 220.2 103) (end 207.2 103) (width 0.25) (layer F.Cu) (net 33))
+  (segment (start 220.2 119.6) (end 220.2 103) (width 0.25) (layer F.Cu) (net 33))
+  (segment (start 220.095 119.705) (end 220.2 119.6) (width 0.25) (layer F.Cu) (net 33))
+  (segment (start 213.9 120.975) (end 220.8 121) (width 0.25) (layer F.Cu) (net 35) (status 400000))
+  (segment (start 208.25 102.35) (end 208.25 96.7) (width 0.25) (layer F.Cu) (net 35) (status 800000))
+  (segment (start 208.2 102.4) (end 208.25 102.35) (width 0.25) (layer F.Cu) (net 35))
+  (segment (start 220.8 102.4) (end 208.2 102.4) (width 0.25) (layer F.Cu) (net 35))
+  (segment (start 220.825 120.975) (end 220.8 102.4) (width 0.25) (layer F.Cu) (net 35))
+  (segment (start 220.8 121) (end 220.825 120.975) (width 0.25) (layer F.Cu) (net 35))
   (segment (start 93 102.95) (end 93 105) (width 0.25) (layer F.Cu) (net 42))
   (segment (start 93.25 105.25) (end 93.25 107.0007) (width 0.25) (layer F.Cu) (net 42))
   (segment (start 93 105) (end 93.25 105.25) (width 0.25) (layer F.Cu) (net 42))
   (segment (start 93.25 107.0007) (end 93 107.2507) (width 0.25) (layer F.Cu) (net 42))
+  (segment (start 214.7 93.75) (end 217.6 93.9) (width 0.25) (layer F.Cu) (net 45) (status 400000))
+  (segment (start 201.815 123.515) (end 201.8 123.5) (width 0.25) (layer F.Cu) (net 45))
+  (via (at 201.8 123.5) (size 0.6) (drill 0.4) (layers F.Cu B.Cu) (net 45))
+  (segment (start 201.8 123.5) (end 201.8 92.9) (width 0.25) (layer B.Cu) (net 45))
+  (segment (start 201.8 92.9) (end 201.8 92.8) (width 0.25) (layer B.Cu) (net 45))
+  (segment (start 201.8 92.8) (end 204.7 92.8) (width 0.25) (layer B.Cu) (net 45))
+  (segment (start 204.7 92.8) (end 212.7 92.8) (width 0.25) (layer B.Cu) (net 45))
+  (segment (start 212.7 92.8) (end 216.1 92.8) (width 0.25) (layer B.Cu) (net 45))
+  (segment (start 216.1 92.8) (end 216.168199 92.868199) (width 0.25) (layer B.Cu) (net 45))
+  (segment (start 216.168199 92.868199) (end 216.368199 92.868199) (width 0.25) (layer B.Cu) (net 45))
+  (segment (start 216.368199 92.868199) (end 216.6 93.1) (width 0.25) (layer B.Cu) (net 45))
+  (segment (start 216.6 93.1) (end 216.9 93.1) (width 0.25) (layer B.Cu) (net 45))
+  (segment (start 216.9 93.1) (end 217 93.1) (width 0.25) (layer B.Cu) (net 45))
+  (segment (start 217 93.1) (end 217.1 93) (width 0.25) (layer B.Cu) (net 45))
+  (segment (start 217.1 93) (end 218.2 92.3) (width 0.25) (layer B.Cu) (net 45))
+  (segment (start 218.2 92.3) (end 219.7 91.75) (width 0.25) (layer B.Cu) (net 45))
+  (segment (start 219.7 91.75) (end 219.8 91.65) (width 0.25) (layer B.Cu) (net 45))
+  (via (at 219.8 91.65) (size 0.6) (drill 0.4) (layers F.Cu B.Cu) (net 45))
+  (segment (start 219.8 91.65) (end 220.1 93.95) (width 0.25) (layer F.Cu) (net 45))
+  (segment (start 220.1 93.95) (end 220.05 94) (width 0.25) (layer F.Cu) (net 45))
+  (segment (start 220.05 94) (end 218 93.9) (width 0.25) (layer F.Cu) (net 45))
+  (segment (start 201.815 123.515) (end 204.5 123.515) (width 0.25) (layer F.Cu) (net 45) (status 800000))
+  (segment (start 217.6 93.9) (end 218 93.9) (width 0.25) (layer F.Cu) (net 45))
+  (segment (start 219 91.5) (end 218.7 91.5) (width 0.25) (layer F.Cu) (net 46))
+  (segment (start 219.5 93.5) (end 219.4 92.3) (width 0.25) (layer F.Cu) (net 46))
+  (segment (start 219.4 92.3) (end 219 91.9) (width 0.25) (layer F.Cu) (net 46))
+  (segment (start 219 91.9) (end 219 91.5) (width 0.25) (layer F.Cu) (net 46))
+  (segment (start 214.7 93.25) (end 219.5 93.5) (width 0.25) (layer F.Cu) (net 46) (status 400000))
+  (segment (start 196.25 86.65) (end 196.25 84.275) (width 0.25) (layer F.Cu) (net 46) (status 800000))
+  (segment (start 196.2 86.7) (end 196.25 86.65) (width 0.25) (layer F.Cu) (net 46))
+  (via (at 196.2 86.7) (size 0.6) (drill 0.4) (layers F.Cu B.Cu) (net 46))
+  (segment (start 218.65 86.7) (end 196.2 86.7) (width 0.25) (layer B.Cu) (net 46))
+  (segment (start 218.65 91.45) (end 218.65 86.7) (width 0.25) (layer B.Cu) (net 46))
+  (via (at 218.65 91.45) (size 0.6) (drill 0.4) (layers F.Cu B.Cu) (net 46))
+  (segment (start 218.7 91.5) (end 218.65 91.45) (width 0.25) (layer F.Cu) (net 46))
+  (segment (start 217.9 93.45) (end 218.05 93.45) (width 0.25) (layer B.Cu) (net 47))
+  (via (at 204.5 127.5) (size 0.6) (drill 0.4) (layers F.Cu B.Cu) (net 47))
+  (segment (start 204.5 127.5) (end 204.5 121.35) (width 0.25) (layer B.Cu) (net 47))
+  (segment (start 204.5 121.35) (end 204.5 93.25) (width 0.25) (layer B.Cu) (net 47))
+  (segment (start 204.5 93.25) (end 209.2 93.25) (width 0.25) (layer B.Cu) (net 47))
+  (segment (start 209.2 93.25) (end 209.200002 93.250002) (width 0.25) (layer B.Cu) (net 47))
+  (segment (start 209.200002 93.250002) (end 215.900002 93.250002) (width 0.25) (layer B.Cu) (net 47))
+  (segment (start 215.900002 93.250002) (end 216.200002 93.550002) (width 0.25) (layer B.Cu) (net 47))
+  (segment (start 216.200002 93.550002) (end 217.799998 93.550002) (width 0.25) (layer B.Cu) (net 47))
+  (segment (start 217.799998 93.550002) (end 217.9 93.45) (width 0.25) (layer B.Cu) (net 47))
+  (segment (start 204.5 126.055) (end 204.5 127.5) (width 0.25) (layer F.Cu) (net 47) (status 400000))
+  (segment (start 218.65 92.75) (end 214.7 92.75) (width 0.25) (layer F.Cu) (net 47) (status 800000))
+  (segment (start 218.7 92.8) (end 218.65 92.75) (width 0.25) (layer F.Cu) (net 47))
+  (via (at 218.7 92.8) (size 0.6) (drill 0.4) (layers F.Cu B.Cu) (net 47))
+  (segment (start 218.05 93.45) (end 218.7 92.8) (width 0.25) (layer B.Cu) (net 47))
   (segment (start 214.7 90.25) (end 226.03 90.25) (width 0.25) (layer F.Cu) (net 48))
   (segment (start 226.03 90.25) (end 226.2 90.42) (width 0.25) (layer F.Cu) (net 48))
@@
   (segment (start 206 79.050002) (end 193.749998 79.050002) (width 0.25) (layer F.Cu) (net 54))
   (segment (start 206.25 79.300002) (end 206 79.050002) (width 0.25) (layer F.Cu) (net 54))
+  (segment (start 213.9 115.895) (end 217.295 115.895) (width 0.25) (layer F.Cu) (net 55) (status 400000))
+  (segment (start 222.35 116.35) (end 222.35 120.7) (width 0.25) (layer B.Cu) (net 55) (status 800000))
+  (segment (start 222 116) (end 222.35 116.35) (width 0.25) (layer B.Cu) (net 55))
+  (segment (start 217.4 116) (end 222 116) (width 0.25) (layer B.Cu) (net 55))
+  (via (at 217.4 116) (size 0.6) (drill 0.4) (layers F.Cu B.Cu) (net 55))
+  (segment (start 217.295 115.895) (end 217.4 116) (width 0.25) (layer F.Cu) (net 55))
+  (segment (start 213.9 114.625) (end 217.975 114.625) (width 0.25) (layer F.Cu) (net 56) (status 400000))
+  (segment (start 218.52 128.32) (end 222.35 128.32) (width 0.25) (layer B.Cu) (net 56) (status 800000))
+  (segment (start 218.4 128.2) (end 218.52 128.32) (width 0.25) (layer B.Cu) (net 56))
+  (segment (start 218.4 117.2) (end 218.4 128.2) (width 0.25) (layer B.Cu) (net 56))
+  (segment (start 218.2 117) (end 218.4 117.2) (width 0.25) (layer B.Cu) (net 56))
+  (via (at 218.2 117) (size 0.6) (drill 0.4) (layers F.Cu B.Cu) (net 56))
+  (segment (start 218.2 114.85) (end 218.2 117) (width 0.25) (layer F.Cu) (net 56))
+  (segment (start 217.975 114.625) (end 218.2 114.85) (width 0.25) (layer F.Cu) (net 56))
+  (segment (start 213.9 113.355) (end 219.155 113.355) (width 0.25) (layer F.Cu) (net 57) (status 400000))
+  (segment (start 219.58 125.78) (end 222.35 125.78) (width 0.25) (layer B.Cu) (net 57) (status 800000))
+  (segment (start 219.4 125.6) (end 219.58 125.78) (width 0.25) (layer B.Cu) (net 57))
+  (segment (start 219.4 116.8) (end 219.4 125.6) (width 0.25) (layer B.Cu) (net 57))
+  (via (at 219.4 116.8) (size 0.6) (drill 0.4) (layers F.Cu B.Cu) (net 57))
+  (segment (start 219.4 113.6) (end 219.4 116.8) (width 0.25) (layer F.Cu) (net 57))
+  (segment (start 219.155 113.355) (end 219.4 113.6) (width 0.25) (layer F.Cu) (net 57))
   (segment (start 84.3 119.555) (end 82.055 119.555) (width 0.25) (layer F.Cu) (net 58))
   (segment (start 81.75 119.25) (end 77 119.25) (width 0.25) (layer B.Cu) (net 58))

Commit message: PCB3 progress: Needs capacitors/resistors and push buttons
Parts:
- moved U6 104.0 mm to (197.2, 98.7), turned to 180 degrees
- moved U7 82.1 mm to (187.1, 101.2)
- moved REF** 1.75 mm to (198.0, 74.8)
Routing:
- net PC0_MP3-SCL: track 0.00 -> 82.5 mm, vias 0 -> 2
- net PC1_MP3-SDA: track 0.00 -> 77.8 mm, vias 0 -> 2
- net PB3_BTpcm-CLK: track 0.00 -> 76.3 mm, vias 0 -> 3
- net PC3_mic: track 0.00 -> 68.7 mm, vias 0 -> 1
- net PB2_BT-GP2: track 0.00 -> 62.6 mm, vias 0 -> 2
- net PB0_BT-GP9: track 0.00 -> 62.3 mm, vias 0 -> 2
- net PB5_BTpcm-IN: track 0.00 -> 61.9 mm, vias 0 -> 2
- net PA4_BTpcm-Sync: track 0.00 -> 54.8 mm, vias 0 -> 1
- net PA6_BT-RTS: track 0.00 -> 52.6 mm, vias 0 -> 2
- net PB1_BT-CTS: track 0.00 -> 49.1 mm, vias 0 -> 2
- net PC5_BT-TX: track 0.00 -> 48.0 mm, vias 0 -> 2
- net PC4_BT-RX: track 0.00 -> 47.8 mm, vias 0 -> 2
- net PB12_MAG-INT: track 0.00 -> 47.1 mm, vias 0 -> 2
- net PA14_dbg: track 0.00 -> 45.2 mm, vias 0 -> 5
- net PA13_dbg: track 19.7 -> 64.2 mm, vias 0 -> 7
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Other:
- board size 95 x 99 mm -> 88 x 91.2 mm
