File: Schematic/Minimal/kicad/_saved_SDMin.sch (KiCad schematic (older format))
At the start: 84 parts, among them CON1 uSD_Card, P1 USB_B, P2 CONN_01X04, P3 CONN_01X04, P4 CONN_01X04, P5 CONN_01X03, P6 CONN_01X03, SW1 SW_PUSH, SW2 SW_PUSH, SW3 SW_PUSH, SW4 SW_PUSH, SW6 SW_PUSH, SW7 SW_PUSH, SW8 SW_PUSH, SW9 SW_PUSH, U1 PAM2301, U10 ADMP401-BB, U11 RN-52, U12 STA013, U2 XC9140, U3 MCP73811/2, U4 STM32L476R, U5 Lightware_SF10/A, U6 UART, U7 DebugPins, U8 MLX90393, U9 LS20031, X1 14.7456MHz

Commit message: Lots of progress on the mPCB
Parts:
- removed D4: D_Schottky_Small, POW:POWERDI-123, symbol D_Schottky_Small
- added C31, C32, C33, C34: 0.1uF, Capacitors_SMD:C_0805_HandSoldering, symbol C_Small
- added R20: 10K, Resistors_SMD:R_0805_HandSoldering, symbol R_Small
- added SW5: SW_PUSH, Buttons_Switches_ThroughHole:SW_PUSH_SMALL, symbol SW_PUSH
- P6: value CONN_01X03 -> CONN_01X02; footprint Socket_Strips:Socket_Strip_Straight_1x03 -> Socket_Strips:Socket_Strip_Straight_1x02; symbol CONN_01X03 -> CONN_01X02
- U7: footprint Pin_Headers:Pin_Header_Straight_1x04 -> Socket_Strips:Socket_Strip_Straight_1x06
Connections:
- net labels removed: x-in-3
- wire segments 268 -> 277
- no-connect marks 34 -> 33
