File: Schematic/Minimal/kicad/fourbis.kicad_pcb (KiCad board)
At the start: 2 copper layers, 75 x 135 mm, 87 parts, among them CON1 uSD_Card, P1 USB_B, P2 CONN_01X04, P3 CONN_01X04, P4 CONN_01X04, P5 CONN_01X03, P6 CONN_01X02, SW1 SW_PUSH, SW2 SW_PUSH, SW3 SW_PUSH, SW4 SW_PUSH, SW5 SW_PUSH, SW6 SW_PUSH, SW7 SW_PUSH, SW8 SW_PUSH, SW9 SW_PUSH, U1 PAM2301, U10 ADMP401-BB, U11 RN-52, U12 STA013, U2 XC9140, U3 MCP73811/2, U4 STM32L476R, U5 Lightware_SF10/A, U6 UART, U7 DebugPins, U8 MLX90393, U9 LS20031, X1 14.7456MHz

Commit message: Lots of progress on the mPCB
Parts:
- removed C31: 0.1uF, Capacitors_SMD:C_0805_HandSoldering
- removed P5: CONN_01X03, Pin_Headers:Pin_Header_Straight_1x03
- removed P6: CONN_01X02, Socket_Strips:Socket_Strip_Straight_1x02
- removed R20: 10K, Resistors_SMD:R_0805_HandSoldering
- C25, C26, R14, R15: moved to F.Cu
- SW5: value SW_PUSH -> Switch_SPDT_x2; footprint Buttons_Switches_ThroughHole:SW_PUSH_SMALL -> Buttons_Switches_ThroughHole:SW_Micro_SPST
- U6: footprint Socket_Strips:Socket_Strip_Straight_1x02 -> Pin_Headers:Pin_Header_Straight_1x02
- U7: footprint Socket_Strips:Socket_Strip_Straight_1x06 -> Pin_Headers:Pin_Header_Straight_1x04
- moved SW5 93.0 mm to (40.5, 155.5), turned to 270 degrees
- moved D1 73.8 mm to (107.0, 80.0), turned to 180 degrees
- moved C27 32.0 mm to (108.0, 46.0), turned to 90 degrees
- moved C28 31.0 mm to (104.0, 46.0), turned to 90 degrees
- moved R16 22.9 mm to (106.0, 50.0), turned to 180 degrees
- moved U6 17.2 mm to (62.0, 88.0), turned to 270 degrees
- moved C11 14.9 mm to (55.0, 161.0)
- moved C2 14.9 mm to (44.0, 156.5), turned to 270 degrees
- moved U7 13.6 mm to (51.0, 51.0), turned to 0 degrees
- moved L2 11.9 mm to (54.0, 148.0), turned to 0 degrees
- moved C25 8.85 mm to (100.0, 53.0), turned to 270 degrees
- moved C5 6.67 mm to (58.0, 67.0), turned to 90 degrees
- moved U1 6.40 mm to (54.0, 152.0), turned to 0 degrees
- moved C15 5.83 mm to (81.0, 63.0)
- moved C14 5.59 mm to (78.0, 62.0), turned to 270 degrees
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Connections:
- BT1 pad 1: +BATT -> Net-(BT1-Pad1)
- C1 pad 1: /3VEN -> +BATT
- C8 pad 1: +BATT -> Net-(BT1-Pad1)
- SW5 pad 1: NRST -> (no net)
- SW5 pad 2: GND -> +BATT
- U1 pad 1: /3VEN -> +BATT
- U1 pad 4: /3VEN -> +BATT
- U10 pad 1: PB0_mic -> PC3_mic
- U11 pad 11: PB11_BT-GP9 -> PB0_BT-GP9
- U2 pad 1: /5VEN -> +BATT
- U3 pad 3: +BATT -> Net-(BT1-Pad1)
- U4 pad 11: (no net) -> PC3_mic
- U4 pad 26: PB0_mic -> PB0_BT-GP9
- U4 pad 30: PB11_BT-GP9 -> Net-(D1-Pad2)
- U4 pad 38: /5VEN -> (no net)
- U4 pad 56: x-in-1 -> (no net)
- U4 pad 58: x-in-2 -> (no net)
- U4 pad 61: Net-(D1-Pad2) -> (no net)
Routing:
- net +BATT: track 67.0 -> 15.9 mm
- net GND: track 43.2 -> 14.3 mm, vias 4 -> 1
- net Net-(C3-Pad2): track 14.8 -> 0.00 mm
- net /3VEN: track 13.7 -> 0.00 mm
- net +5V: track 12.1 -> 0.00 mm
- net Net-(L2-Pad1): track 9.66 -> 0.00 mm
- net +3V3: track 7.74 -> 0.00 mm
- net Net-(L1-Pad2): track 3.45 -> 0.00 mm
