File: Schematic/Minimal/kicad/endlesscopies/noname14.kicad_pcb (KiCad board)
At the start: 4 copper layers, 75 x 135 mm, 89 parts, among them CON1 uSD_Card, P1 USB_B, P2 CONN_01X04, P3 CONN_01X04, P4 CONN_01X04, P5 CONN_01X03, P6 CONN_01X02, SW1 SW_PUSH, SW2 SW_PUSH, SW3 SW_PUSH, SW4 SW_PUSH, SW5 SW_PUSH, SW6 SW_PUSH, SW7 SW_PUSH, SW8 SW_PUSH, SW9 SW_PUSH, U1 PAM2301, U10 ADMP401-BB, U11 RN-52, U12 STA013, U2 XC9140, U3 MCP73811/2, U4 STM32L476R, U5 Lightware_SF10/A, U6 UART, U7 DebugPins, U8 MLX90393, U9 LS20031, X1 14.7456MHz

Commit message: PCB4-23
Parts:
- moved C14 9.95 mm to (77.5, 51.4)
- moved C15 8.73 mm to (79.7, 52.8)
- moved C6 3.61 mm to (54.0, 64.0)
- moved C13 3.58 mm to (70.0, 79.0)
- moved C5 3.20 mm to (51.5, 65.5)
- moved C10 3.00 mm to (63.0, 79.0)
- moved C9 3.00 mm to (64.0, 81.5)
- moved C12 2.70 mm to (71.0, 81.5)
- moved P4 2.35 mm to (83.8, 84.3)
- moved P2 2.35 mm to (88.9, 84.3)
- moved P3 2.35 mm to (86.4, 84.3)
- moved C16 1.12 mm to (64.2, 51.4)
- moved C17 1.00 mm to (65.5, 53.5)
- moved C4 0.79 mm to (57.2, 59.2), turned to 270 degrees
- moved C20 0.29 mm to (52.0, 75.5), turned to 0 degrees
Routing:
- net GND: track 97.0 -> 417.0 mm, vias 4 -> 14
- net +3V3: track 7.71 -> 311.4 mm, vias 0 -> 2
- net +BATT: track 60.3 -> 55.7 mm, vias 1 -> 0
- net /5VEN: track 0.00 -> 1.05 mm, vias 0 -> 1
- added copper zone on F.Cu, net +3V3
- added copper zone on B.Cu, net GND
- removed copper zone on In2.Cu, net +3V3
- removed copper zone on In1.Cu, net GND
Other:
- copper layers 4 -> 2
