File: Schematic/Minimal/kicad/endlesscopies/noname17.kicad_pcb (KiCad board)
At the start: 4 copper layers, 75 x 135 mm, 89 parts, among them CON1 uSD_Card, P1 USB_B, P2 CONN_01X04, P3 CONN_01X04, P4 CONN_01X04, P5 CONN_01X03, P6 CONN_01X02, SW1 SW_PUSH, SW2 SW_PUSH, SW3 SW_PUSH, SW4 SW_PUSH, SW5 SW_PUSH, SW6 SW_PUSH, SW7 SW_PUSH, SW8 SW_PUSH, SW9 SW_PUSH, U1 PAM2301, U10 ADMP401-BB, U11 RN-52, U12 STA013, U2 XC9140, U3 MCP73811/2, U4 STM32L476R, U5 Lightware_SF10/A, U6 UART, U7 DebugPins, U8 MLX90393, U9 LS20031, X1 14.7456MHz

Commit message: PCB4-23
Parts:
- added D4: D_Small, Diodes_SMD:SOD-523, B.Cu at (44.5, 152.8)
- moved C9 9.01 mm to (63.5, 83.0)
- moved C12 8.81 mm to (72.0, 82.8)
- moved C14 8.66 mm to (77.5, 51.4)
- moved C15 8.20 mm to (79.7, 52.8)
- moved C5 7.76 mm to (51.5, 65.5)
- moved C16 4.75 mm to (64.2, 51.4)
- moved C10 4.00 mm to (62.5, 80.5)
- moved C13 3.78 mm to (71.0, 80.2)
- moved C6 3.20 mm to (54.0, 64.0)
- moved P4 2.35 mm to (83.8, 84.3)
- moved P2 2.35 mm to (88.9, 84.3)
- moved P3 2.35 mm to (86.4, 84.3)
- moved C4 1.46 mm to (57.2, 59.2), turned to 270 degrees
- moved C17 1.00 mm to (65.5, 53.5)
- moved C20 0.29 mm to (52.0, 75.5), turned to 0 degrees
Connections:
- U4 pad 38: /5VEN -> Net-(D4-Pad2)
Routing:
- net GND: track 0.00 -> 431.6 mm, vias 0 -> 15
- net +3V3: track 0.00 -> 347.1 mm, vias 0 -> 1
- net +BATT: track 0.00 -> 55.7 mm
- net Net-(C3-Pad2): track 0.00 -> 14.5 mm
- net /3VEN: track 0.00 -> 12.2 mm
- net Net-(L2-Pad1): track 0.00 -> 7.49 mm
- net +5V: track 0.00 -> 7.38 mm
- net Net-(L1-Pad2): track 0.00 -> 4.50 mm
- net /5VEN: track 0.00 -> 1.94 mm, vias 0 -> 1
- removed copper zone on In2.Cu, net +3V3
- removed copper zone on In1.Cu, net GND
Other:
- copper layers 4 -> 2
