File: Schematic/Minimal/kicad/endlesscopies/noname19-back2wirewrapping.kicad_pcb (KiCad board)
At the start: 4 copper layers, 75 x 135 mm, 89 parts, among them CON1 uSD_Card, P1 USB_B, P2 CONN_01X04, P3 CONN_01X04, P4 CONN_01X04, P5 CONN_01X03, P6 CONN_01X02, SW1 SW_PUSH, SW2 SW_PUSH, SW3 SW_PUSH, SW4 SW_PUSH, SW5 SW_PUSH, SW6 SW_PUSH, SW7 SW_PUSH, SW8 SW_PUSH, SW9 SW_PUSH, U1 PAM2301, U10 ADMP401-BB, U11 RN-52, U12 STA013, U2 XC9140, U3 MCP73811/2, U4 STM32L476R, U5 Lightware_SF10/A, U6 UART, U7 DebugPins, U8 MLX90393, U9 LS20031, X1 14.7456MHz

Commit message: PCB4-23
Parts:
- moved C5 4.00 mm to (55.0, 67.5)
- moved C14 3.72 mm to (80.7, 60.4)
- moved C16 3.61 mm to (63.2, 52.4)
- moved C9 3.50 mm to (64.0, 77.5)
- moved C12 3.29 mm to (72.5, 77.2)
- moved C13 1.75 mm to (71.5, 74.8)
- moved C10 1.58 mm to (63.0, 75.0)
- moved C15 1.58 mm to (78.0, 61.5)
- moved C17 1.50 mm to (64.5, 55.0)
- moved C6 1.50 mm to (58.0, 66.0)
- moved C4 0.71 mm to (58.5, 60.0)
Routing:
- net GND: track 0.00 -> 101.7 mm, vias 0 -> 5
- net +BATT: track 0.00 -> 60.3 mm, vias 0 -> 1
- net Net-(C3-Pad2): track 0.00 -> 14.5 mm
- net /3VEN: track 0.00 -> 12.2 mm
- net Net-(L2-Pad1): track 0.00 -> 7.49 mm
- net +3V3: track 0.00 -> 7.46 mm
- net +5V: track 0.00 -> 7.38 mm
- net Net-(L1-Pad2): track 0.00 -> 4.50 mm
- added copper zone on F.Cu, net +3V3
- added copper zone on B.Cu, net GND
- removed copper zone on In2.Cu, net +3V3
- removed copper zone on In1.Cu, net GND
Other:
- copper layers 4 -> 2
