File: Schematic/Minimal/kicad/endlesscopies/noname22-allauto.kicad_pcb (KiCad board)
At the start: 4 copper layers, 75 x 135 mm, 89 parts, among them CON1 uSD_Card, P1 USB_B, P2 CONN_01X04, P3 CONN_01X04, P4 CONN_01X04, P5 CONN_01X03, P6 CONN_01X02, SW1 SW_PUSH, SW2 SW_PUSH, SW3 SW_PUSH, SW4 SW_PUSH, SW5 SW_PUSH, SW6 SW_PUSH, SW7 SW_PUSH, SW8 SW_PUSH, SW9 SW_PUSH, U1 PAM2301, U10 ADMP401-BB, U11 RN-52, U12 STA013, U2 XC9140, U3 MCP73811/2, U4 STM32L476R, U5 Lightware_SF10/A, U6 UART, U7 DebugPins, U8 MLX90393, U9 LS20031, X1 14.7456MHz

Commit message: PCB4-23
Parts:
- moved C12 5.27 mm to (72.5, 79.2)
- moved C5 5.00 mm to (54.0, 67.5)
- moved C14 4.71 mm to (81.7, 60.4)
- moved C16 4.60 mm to (63.2, 51.4)
- moved C9 4.50 mm to (64.0, 78.5)
- moved C13 0.75 mm to (71.5, 75.8)
- moved C10 0.71 mm to (63.0, 76.0)
- moved C15 0.71 mm to (79.0, 61.5)
- moved C17 0.50 mm to (64.5, 54.0)
- moved C6 0.50 mm to (57.0, 66.0)
Changed lines of the file:
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@@
   (general
     (links 273)
-    (no_connects 232)
+    (no_connects 273)
     (area 36.924999 39.924999 115.275001 175.075001)
     (thickness 1.6)
@@
   )
   (setup
-    (last_trace_width 0.4)
+    (last_trace_width 0.25)
     (user_trace_width 0.4)
     (user_trace_width 0.5)
@@
   )
   (module Capacitors_ThroughHole:C_Radial_D5_L11_P2.5 (layer F.Cu)
-    (at 56.5 66 270)
+    (at 57 66 270)
     (descr "Radial Electrolytic Capacitor Diameter 5mm x Length 11mm, Pitch 2.5mm")
     (tags "Electrolytic Capacitor")
@@
   )
   (module Capacitors_ThroughHole:C_Radial_D5_L11_P2.5 (layer F.Cu)
-    (at 62.5 76.5)
+    (at 63 76)
     (descr "Radial Electrolytic Capacitor Diameter 5mm x Length 11mm, Pitch 2.5mm")
     (tags "Electrolytic Capacitor")
@@
   )
   (module Capacitors_ThroughHole:C_Radial_D5_L11_P2.5 (layer F.Cu)
-    (at 64.5 53.5 180)
+    (at 64.5 54 180)
     (descr "Radial Electrolytic Capacitor Diameter 5mm x Length 11mm, Pitch 2.5mm")
     (tags "Electrolytic Capacitor")
@@
   )
   (module Capacitors_SMD:C_0805_HandSoldering (layer B.Cu)
-    (at 59 67.5 270)
+    (at 54 67.5 270)
     (descr "Capacitor SMD 0805, hand soldering")
     (tags "capacitor 0805")
@@
   )
   (module Capacitors_SMD:C_0805_HandSoldering (layer B.Cu)
-    (at 64 74)
+    (at 64 78.5)
     (descr "Capacitor SMD 0805, hand soldering")
     (tags "capacitor 0805")
@@
   )
   (module Capacitors_SMD:C_0805_HandSoldering (layer B.Cu)
-    (at 73 74)
+    (at 72.5 79.25)
     (descr "Capacitor SMD 0805, hand soldering")
     (tags "capacitor 0805")
@@
   )
   (module Capacitors_ThroughHole:C_Radial_D5_L11_P2.5 (layer F.Cu)
-    (at 71.5 76.5)
+    (at 71.5 75.75)
     (descr "Radial Electrolytic Capacitor Diameter 5mm x Length 11mm, Pitch 2.5mm")
     (tags "Electrolytic Capacitor")
@@
   )
   (module Capacitors_SMD:C_0805_HandSoldering (layer B.Cu)
-    (at 77 60 90)
+    (at 81.7 60.35 90)
     (descr "Capacitor SMD 0805, hand soldering")
     (tags "capacitor 0805")
@@
   )
   (module Capacitors_ThroughHole:C_Radial_D5_L11_P2.5 (layer F.Cu)
-    (at 79.5 61 90)
+    (at 79 61.5 90)
     (descr "Radial Electrolytic Capacitor Diameter 5mm x Length 11mm, Pitch 2.5mm")
     (tags "Electrolytic Capacitor")
@@
   )
   (module Capacitors_SMD:C_0805_HandSoldering (layer B.Cu)
-    (at 63 56 180)
+    (at 63.2 51.4 180)
     (descr "Capacitor SMD 0805, hand soldering")
     (tags "capacitor 0805")
@@
     (polygon
       (pts
+        (xy 74.75 80.25) (xy 70.25 80.25) (xy 70.25 78.25) (xy 74.75 78.25) (xy 74.75 80.25)
+      )
+    )
+  )
+  (zone (net 0) (net_name "") (layer B.Cu) (hatch edge 0.508)
+    (connect_pads (clearance 0.508))
+    (min_thickness 0.254)
+    (keepout (tracks allowed) (vias not_allowed) (copperpour allowed))
+    (fill (arc_segments 16) (thermal_gap 0.508) (thermal_bridge_width 0.508))
+    (polygon
+      (pts
+        (xy 74.75 80.25) (xy 70.25 80.25) (xy 70.25 78.25) (xy 74.75 78.25) (xy 74.75 80.25)
+      )
+    )
+  )
+  (zone (net 0) (net_name "") (layer B.Cu) (hatch edge 0.508)
+    (connect_pads (clearance 0.508))
+    (min_thickness 0.254)
+    (keepout (tracks allowed) (vias not_allowed) (copperpour allowed))
+    (fill (arc_segments 16) (thermal_gap 0.508) (thermal_bridge_width 0.508))
+    (polygon
+      (pts
+        (xy 66.25 79.5) (xy 61.75 79.5) (xy 61.75 77.5) (xy 66.25 77.5) (xy 66.25 79.5)
+      )
+    )
+  )
+  (zone (net 0) (net_name "") (layer F.Cu) (hatch edge 0.508)
+    (connect_pads (clearance 0.508))
+    (min_thickness 0.254)
+    (keepout (tracks allowed) (vias not_allowed) (copperpour allowed))
+    (fill (arc_segments 16) (thermal_gap 0.508) (thermal_bridge_width 0.508))
+    (polygon
+      (pts
+        (xy 66.25 79.5) (xy 61.75 79.5) (xy 61.75 77.5) (xy 66.25 77.5) (xy 66.25 79.5)
+      )
+    )
+  )
+  (zone (net 0) (net_name "") (layer F.Cu) (hatch edge 0.508)
+    (connect_pads (clearance 0.508))
+    (min_thickness 0.254)
+    (keepout (tracks allowed) (vias not_allowed) (copperpour allowed))
+    (fill (arc_segments 16) (thermal_gap 0.508) (thermal_bridge_width 0.508))
+    (polygon
+      (pts
+        (xy 55 69.75) (xy 53 69.75) (xy 53 65.25) (xy 55 65.25) (xy 55 69.75)
+      )
+    )
+  )
+  (zone (net 0) (net_name "") (layer B.Cu) (hatch edge 0.508)
+    (connect_pads (clearance 0.508))
+    (min_thickness 0.254)
+    (keepout (tracks allowed) (vias not_allowed) (copperpour allowed))
+    (fill (arc_segments 16) (thermal_gap 0.508) (thermal_bridge_width 0.508))
+    (polygon
+      (pts
+        (xy 55 69.75) (xy 53 69.75) (xy 53 65.25) (xy 55 65.25) (xy 55 69.75)
+      )
+    )
+  )
+  (zone (net 0) (net_name "") (layer B.Cu) (hatch edge 0.508)
+    (connect_pads (clearance 0.508))
+    (min_thickness 0.254)
+    (keepout (tracks allowed) (vias not_allowed) (copperpour allowed))
+    (fill (arc_segments 16) (thermal_gap 0.508) (thermal_bridge_width 0.508))
+    (polygon
+      (pts
+        (xy 60.25 61.5) (xy 55.75 61.5) (xy 55.75 59.5) (xy 60.25 59.5) (xy 60.25 61.5)
+      )
+    )
+  )
+  (zone (net 0) (net_name "") (layer F.Cu) (hatch edge 0.508)
+    (connect_pads (clearance 0.508))
+    (min_thickness 0.254)
+    (keepout (tracks allowed) (vias not_allowed) (copperpour allowed))
+    (fill (arc_segments 16) (thermal_gap 0.508) (thermal_bridge_width 0.508))
+    (polygon
+      (pts
+        (xy 60.25 61.5) (xy 55.75 61.5) (xy 55.75 59.5) (xy 60.25 59.5) (xy 60.25 61.5)
+      )
+    )
+  )
+  (zone (net 0) (net_name "") (layer F.Cu) (hatch edge 0.508)
+    (connect_pads (clearance 0.508))
+    (min_thickness 0.254)
+    (keepout (tracks allowed) (vias not_allowed) (copperpour allowed))
+    (fill (arc_segments 16) (thermal_gap 0.508) (thermal_bridge_width 0.508))
+    (polygon
+      (pts
+        (xy 65.45 52.4) (xy 60.95 52.4) (xy 60.95 50.4) (xy 65.45 50.4) (xy 65.45 52.4)
+      )
+    )
+  )
+  (zone (net 0) (net_name "") (layer B.Cu) (hatch edge 0.508)
+    (connect_pads (clearance 0.508))
+    (min_thickness 0.254)
+    (keepout (tracks allowed) (vias not_allowed) (copperpour allowed))
+    (fill (arc_segments 16) (thermal_gap 0.508) (thermal_bridge_width 0.508))
+    (polygon
+      (pts
+        (xy 65.45 52.4) (xy 60.95 52.4) (xy 60.95 50.4) (xy 65.45 50.4) (xy 65.45 52.4)
+      )
+    )
+  )
+  (zone (net 0) (net_name "") (layer F.Cu) (hatch edge 0.508)
+    (connect_pads (clearance 0.508))
+    (min_thickness 0.254)
+    (keepout (tracks allowed) (vias not_allowed) (copperpour allowed))
+    (fill (arc_segments 16) (thermal_gap 0.508) (thermal_bridge_width 0.508))
+    (polygon
+      (pts
+        (xy 82.7 62.6) (xy 80.7 62.6) (xy 80.7 58.1) (xy 82.7 58.1) (xy 82.7 62.6)
+      )
+    )
+  )
+  (zone (net 0) (net_name "") (layer B.Cu) (hatch edge 0.508)
+    (connect_pads (clearance 0.508))
+    (min_thickness 0.254)
+    (keepout (tracks allowed) (vias not_allowed) (copperpour allowed))
+    (fill (arc_segments 16) (thermal_gap 0.508) (thermal_bridge_width 0.508))
+    (polygon
+      (pts
+        (xy 82.7 62.6) (xy 80.7 62.6) (xy 80.7 58.1) (xy 82.7 58.1) (xy 82.7 62.6)
+      )
+    )
+  )
+  (zone (net 0) (net_name "") (layer F.Cu) (hatch edge 0.508)
+    (connect_pads (clearance 0.508))
+    (min_thickness 0.254)
+    (keepout (tracks allowed) (vias not_allowed) (copperpour allowed))
+    (fill (arc_segments 16) (thermal_gap 0.508) (thermal_bridge_width 0.508))
+    (polygon
+      (pts
         (xy 50 74.35) (xy 54.5 74.35) (xy 54.5 76.35) (xy 50 76.35) (xy 50 74.35)
       )
@@
     )
   )
-  (zone (net 1) (net_name GND) (layer In1.Cu) (hatch edge 0.508)
+  (zone (net 4) (net_name +3V3) (layer In2.Cu) (hatch edge 0.508)
     (connect_pads (clearance 0.508))
     (min_thickness 0.254)
-    (fill yes (arc_segments 16) (thermal_gap 0.508) (thermal_bridge_width 0.508))
+    (fill (arc_segments 16) (thermal_gap 0.508) (thermal_bridge_width 0.508))
     (polygon
       (pts
-        (xy 111 174) (xy 38 174) (xy 38 41) (xy 111 41) (xy 111 174)
+        (xy 111.5 174.5) (xy 37.5 174.5) (xy 37.5 40.5) (xy 111.5 40.5) (xy 111.5 174.5)
       )
     )
   )
-  (zone (net 4) (net_name +3V3) (layer In2.Cu) (hatch edge 0.508)
+  (zone (net 1) (net_name GND) (layer In1.Cu) (hatch edge 0.508)
     (connect_pads (clearance 0.508))
     (min_thickness 0.254)
-    (fill yes (arc_segments 16) (thermal_gap 0.508) (thermal_bridge_width 0.508))
+    (fill (arc_segments 16) (thermal_gap 0.508) (thermal_bridge_width 0.508))
     (polygon
       (pts
-        (xy 111 174) (xy 38 174) (xy 38 41) (xy 111 41) (xy 111 174)
+        (xy 111.5 174.5) (xy 37.5 174.5) (xy 37.5 40.5) (xy 111.5 40.5) (xy 111.5 174.5)
       )
     )
