File: Schematic/Minimal/kicad/endlesscopies/_autosave-noname22-allauto.kicad_pcb (KiCad board)
At the start: 4 copper layers, 75 x 135 mm, 89 parts, among them CON1 uSD_Card, P1 USB_B, P2 CONN_01X04, P3 CONN_01X04, P4 CONN_01X04, P5 CONN_01X03, P6 CONN_01X02, SW1 SW_PUSH, SW2 SW_PUSH, SW3 SW_PUSH, SW4 SW_PUSH, SW5 SW_PUSH, SW6 SW_PUSH, SW7 SW_PUSH, SW8 SW_PUSH, SW9 SW_PUSH, U1 PAM2301, U10 ADMP401-BB, U11 RN-52, U12 STA013, U2 XC9140, U3 MCP73811/2, U4 STM32L476R, U5 Lightware_SF10/A, U6 UART, U7 DebugPins, U8 MLX90393, U9 LS20031, X1 14.7456MHz

Commit message: PCB4:25
Parts:
- moved C5 5.00 mm to (54.0, 67.5)
- moved C14 4.78 mm to (81.7, 60.4)
- moved C12 4.78 mm to (72.5, 79.2)
- moved C16 4.60 mm to (63.2, 51.4)
- moved C9 4.50 mm to (64.0, 78.5)
- moved C13 1.25 mm to (71.5, 75.8)
- moved C15 1.12 mm to (79.0, 61.5)
- moved C10 0.71 mm to (63.0, 76.0)
- moved C17 0.50 mm to (64.5, 54.0)
- moved C6 0.50 mm to (57.0, 66.0)
Routing:
- net /in6: track 0.00 -> 149.6 mm, vias 0 -> 1
- net /in7: track 0.00 -> 139.3 mm, vias 0 -> 1
- net PB7_GPS-TX: track 0.00 -> 138.4 mm, vias 0 -> 1
- net /in1: track 0.00 -> 134.9 mm
- net GND: track 0.00 -> 128.9 mm, vias 0 -> 51
- net /in8: track 0.00 -> 126.3 mm, vias 0 -> 1
- net /in3: track 0.00 -> 116.8 mm
- net /in4: track 0.00 -> 107.2 mm
- net +5V: track 0.00 -> 106.6 mm
- net PA7_MP3-SDI: track 0.00 -> 102.6 mm, vias 0 -> 2
- net /5VEN: track 0.00 -> 102.5 mm
- net +3V3: track 0.00 -> 99.3 mm, vias 0 -> 35
- net PD2_SD-CMD: track 0.00 -> 97.4 mm, vias 0 -> 2
- net PC11_SD-D3: track 0.00 -> 96.9 mm, vias 0 -> 2
- net /in2: track 0.00 -> 94.9 mm, vias 0 -> 1
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