File: Schematic/Minimal/kicad/endlesscopies/noname24-flippedcaps.kicad_pcb (KiCad board)
At the start: 4 copper layers, 75 x 135 mm, 89 parts, among them CON1 uSD_Card, P1 USB_B, P2 CONN_01X04, P3 CONN_01X04, P4 CONN_01X04, P5 CONN_01X03, P6 CONN_01X02, SW1 SW_PUSH, SW2 SW_PUSH, SW3 SW_PUSH, SW4 SW_PUSH, SW5 SW_PUSH, SW6 SW_PUSH, SW7 SW_PUSH, SW8 SW_PUSH, SW9 SW_PUSH, U1 PAM2301, U10 ADMP401-BB, U11 RN-52, U12 STA013, U2 XC9140, U3 MCP73811/2, U4 STM32L476R, U5 Lightware_SF10/A, U6 UART, U7 DebugPins, U8 MLX90393, U9 LS20031, X1 14.7456MHz

Commit message: PCB4:25
Parts:
- C12, C14, C16, C5, C9: moved to F.Cu
- moved C12 0.50 mm to (73.0, 74.0)
- moved C13 0.50 mm to (71.5, 76.5)
- moved C14 0.50 mm to (77.0, 60.0)
- moved C15 0.50 mm to (79.5, 61.0)
