File: Schematic/Minimal/kicad/endlesscopies/noname26.kicad_pcb (KiCad board)
At the start: 4 copper layers, 75 x 135 mm, 89 parts, among them CON1 uSD_Card, P1 USB_B, P2 CONN_01X04, P3 CONN_01X04, P4 CONN_01X04, P5 CONN_01X03, P6 CONN_01X02, SW1 SW_PUSH, SW2 SW_PUSH, SW3 SW_PUSH, SW4 SW_PUSH, SW5 SW_PUSH, SW6 SW_PUSH, SW7 SW_PUSH, SW8 SW_PUSH, SW9 SW_PUSH, U1 PAM2301, U10 ADMP401-BB, U11 RN-52, U12 STA013, U2 XC9140, U3 MCP73811/2, U4 STM32L476R, U5 Lightware_SF10/A, U6 UART, U7 DebugPins, U8 MLX90393, U9 LS20031, X1 14.7456MHz

Commit message: PCB svg render
Routing:
- net /in6: track 0.00 -> 154.2 mm, vias 0 -> 1
- net /in1: track 0.00 -> 137.0 mm
- net /in7: track 0.00 -> 131.9 mm
- net GND: track 0.00 -> 127.2 mm, vias 0 -> 50
- net /in8: track 0.00 -> 126.0 mm, vias 0 -> 1
- net PB7_GPS-TX: track 0.00 -> 125.0 mm, vias 0 -> 1
- net /in3: track 0.00 -> 117.0 mm
- net /in4: track 0.00 -> 107.5 mm
- net +3V3: track 0.00 -> 106.5 mm, vias 0 -> 31
- net +5V: track 0.00 -> 106.2 mm
- net /5VEN: track 0.00 -> 102.0 mm, vias 0 -> 2
- net /in5: track 0.00 -> 95.5 mm, vias 0 -> 1
- net PC8_SD-D0: track 0.00 -> 91.2 mm, vias 0 -> 2
- net /in2: track 0.00 -> 90.9 mm, vias 0 -> 1
- net PC11_SD-D3: track 0.00 -> 87.1 mm, vias 0 -> 2
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